File: hardware/boards/main-control-board/main-control-board-esp32.kicad_sch (KiCad schematic)
At the start: 3 parts, among them J7 Conn_ESP32_L, J8 Conn_ESP32_R

Commit message: set FT Rotation Offset to fix JLCPCB orientation
Parts:
- J7, J8: FT Rotation Offset (none) -> 90
Changed lines of the file:
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@@
+			)
+		)
+		(property "FT Rotation Offset" "90"
+			(at 99.06 54.61 90)
+			(hide yes)
+			(show_name no)
+			(do_not_autoplace no)
+			(effects
+				(font
+					(size 1.27 1.27)
+				)
 			)
 		)
@@
 			(at 177.8 54.61 90)
 			(hide yes)
+			(show_name no)
+			(do_not_autoplace no)
+			(effects
+				(font
+					(size 1.27 1.27)
+				)
+			)
+		)
+		(property "FT Rotation Offset" "90"
+			(at 177.8 54.61 90)
+			(hide yes)

Commit message: integrate PCA into the board
Parts:
- J7, J8: FT Rotation Offset 90 -> (none)
Changed lines of the file:
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@@
-			)
-		)
-		(property "FT Rotation Offset" "90"
-			(at 99.06 54.61 90)
-			(hide yes)
-			(show_name no)
-			(do_not_autoplace no)
-			(effects
-				(font
-					(size 1.27 1.27)
-				)
 			)
 		)
@@
 			(at 177.8 54.61 90)
 			(hide yes)
-			(show_name no)
-			(do_not_autoplace no)
-			(effects
-				(font
-					(size 1.27 1.27)
-				)
-			)
-		)
-		(property "FT Rotation Offset" "90"
-			(at 177.8 54.61 90)
-			(hide yes)
