File: hardware/boards/main-control-board/main-control-board-esp32.kicad_sch (KiCad schematic)
At the start: 3 parts, among them J7 Conn_ESP32_L, J8 Conn_ESP32_R

Commit message: turn test points into extension points
Connections:
- net GP6: now reaches ESP2.10 (GP6), J8.1 (Pin_1)
Changed lines of the file:
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@@
+	)
+	(junction
+		(at 167.64 95.25)
+		(diameter 0)
+		(color 0 0 0 0)
 	)
 	(junction
@@
 		(pts
 			(xy 96.52 82.55) (xy 119.38 82.55)
+		)
+		(stroke
+			(width 0)
+			(type default)
+		)
+	)
+	(wire
+		(pts
+			(xy 167.64 95.25) (xy 194.31 95.25)
 		)
 		(stroke
@@
 		)
 	)
+	(hierarchical_label "GP6"
+		(shape input)
+		(at 194.31 95.25 0)
+		(effects
+			(font
+				(size 1.27 1.27)
+			)
+			(justify left)
+		)
+	)

Commit message: pre-fab improvements
Connections:
- net UDB_DP renamed USB_DP
Changed lines of the file:
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@@
 		)
 	)
-	(hierarchical_label "UDB_DP"
-		(shape input)
+	(hierarchical_label "USB_DP"
+		(shape bidirectional)
 		(at 194.31 80.01 0)
 		(effects
@@
 	)
 	(hierarchical_label "GP1"
-		(shape input)
+		(shape bidirectional)
 		(at 88.9 85.09 180)
 		(effects
@@
 	)
 	(hierarchical_label "GP5"
-		(shape input)
+		(shape bidirectional)
 		(at 88.9 95.25 180)
 		(effects
@@
 	)
 	(hierarchical_label "GP6"
-		(shape input)
+		(shape bidirectional)
 		(at 194.31 95.25 0)
 		(effects
@@
 	)
 	(hierarchical_label "GP0"
-		(shape input)
+		(shape bidirectional)
 		(at 88.9 82.55 180)
 		(effects
@@
 	)
 	(hierarchical_label "GP2"
-		(shape input)
+		(shape bidirectional)
 		(at 88.9 87.63 180)
 		(effects
@@
 	)
 	(hierarchical_label "GP3"
-		(shape input)
+		(shape bidirectional)
 		(at 88.9 90.17 180)
 		(effects
@@
 	)
 	(hierarchical_label "GP4"
-		(shape input)
+		(shape bidirectional)
 		(at 88.9 92.71 180)
 		(effects
@@
 	)
 	(hierarchical_label "USB_DM"
-		(shape input)
+		(shape bidirectional)
 		(at 194.31 82.55 0)
 		(effects

Commit message: feat(pcb): update component properties and add missing attributes
- Renamed connection values for ESP32 components to standardize naming.
- Added properties for KiLib_Generator, MPN, and Manufacturer for various components across multiple schematic files.
- Enhanced documentation for component attributes to improve clarity and accessibility in the design process.
Parts:
- J7: value Conn_ESP32_L -> Conn_ESP32; MPN (none) -> PM254-1-09-Z-8.5; Manufacturer (none) -> HCTL
- J8: value Conn_ESP32_R -> Conn_ESP32; MPN (none) -> PM254-1-09-Z-8.5; Manufacturer (none) -> HCTL
Changed lines of the file:
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@@
 			)
 		)
-		(property "Value" "Conn_ESP32_L"
+		(property "Value" "Conn_ESP32"
 			(at 99.06 52.07 90)
 			(show_name no)
@@
 		)
 		(property "FT Rotation Offset" "90"
+			(at 99.06 54.61 90)
+			(hide yes)
+			(show_name no)
+			(do_not_autoplace no)
+			(effects
+				(font
+					(size 1.27 1.27)
+				)
+			)
+		)
+		(property "KiLib_Generator" ""
+			(at 99.06 54.61 90)
+			(hide yes)
+			(show_name no)
+			(do_not_autoplace no)
+			(effects
+				(font
+					(size 1.27 1.27)
+				)
+			)
+		)
+		(property "MPN" "PM254-1-09-Z-8.5"
+			(at 99.06 54.61 90)
+			(hide yes)
+			(show_name no)
+			(do_not_autoplace no)
+			(effects
+				(font
+					(size 1.27 1.27)
+				)
+			)
+		)
+		(property "Manufacturer" "HCTL"
 			(at 99.06 54.61 90)
 			(hide yes)
@@
 			)
 		)
-		(property "Value" "Conn_ESP32_R"
+		(property "Value" "Conn_ESP32"
 			(at 177.8 52.07 90)
 			(show_name no)
@@
 		)
 		(property "FT Rotation Offset" "90"
+			(at 177.8 54.61 90)
+			(hide yes)
+			(show_name no)
+			(do_not_autoplace no)
+			(effects
+				(font
+					(size 1.27 1.27)
+				)
+			)
+		)
+		(property "KiLib_Generator" ""
+			(at 177.8 54.61 90)
+			(hide yes)
+			(show_name no)
+			(do_not_autoplace no)
+			(effects
+				(font
+					(size 1.27 1.27)
+				)
+			)
+		)
+		(property "MPN" "PM254-1-09-Z-8.5"
+			(at 177.8 54.61 90)
+			(hide yes)
+			(show_name no)
+			(do_not_autoplace no)
+			(effects
+				(font
+					(size 1.27 1.27)
+				)
+			)
+		)
+		(property "Manufacturer" "HCTL"
 			(at 177.8 54.61 90)
 			(hide yes)
@@
 			(at 137.16 85.09 0)
 			(hide yes)
+			(show_name no)
+			(do_not_autoplace no)
+			(effects
+				(font
+					(size 1.27 1.27)
+				)
+			)
+		)
+		(property "KiLib_Generator" ""
+			(at 137.16 85.09 0)
+			(hide yes)
